File: STS1_RF.sch (KiCad schematic (older format))
At the start: 22 parts, among them J39 Conn_Coaxial, J40 Conn_Coaxial, J57 Conn_01x01_Male, J58 Conn_01x01_Male, J59 Conn_01x01_Male, J60 Conn_01x01_Male, J61 Conn_01x01_Male, J62 Conn_01x01_Male, J65 Conn_01x02_Male, J66 Conn_01x02_Male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

Commit message: final version1
Parts:
- removed J57, J58, J59, J60, J61, J62: Conn_01x01_Male, Connector_PinHeader_2.54mm:PinHeader_1x01_P2.54mm_Vertical, symbol Connector:Conn_01x01_Male
- removed J65, J66, J67, J68, J69, J70: Conn_01x02_Male, Connector_PinHeader_2.54mm:PinHeader_1x02_P2.54mm_Vertical, symbol Connector:Conn_01x02_Male
- added J10, J11, J7, J8: Conn_01x03_Male, STS1library:PinHeader_1x03_P2.54mm_Vertical_umdieEcke, symbol Connector:Conn_01x03_Male
Connections:
- net GND: now also J10.1 (Pin_1), J11.1 (Pin_1), J7.1 (Pin_1), J8.1 (Pin_1); no longer RF1.12 (NC), RF1.3 (NC), RF1.4 (NC), RF2.14 (NC), RF2.3 (NC), RF2.4 (NC)
- net LoRa_VCC: now also J7.3 (Pin_3), J8.3 (Pin_3)
- net at RF1.13 (DIO1): now also J7.2 (Pin_2)
- net at RF1.14 (DIO3): now also J8.2 (Pin_2)
- net LoRa_NRESET: now reaches RF1.5 (NRESET)
- net at RF2.12 (GPIO1): now also J11.2 (Pin_2)
- net at RF2.13 (GPIO0): now also J10.2 (Pin_2)
- net RF4463F30_SDN: now reaches RF2.5 (SDN)
- new net RF4463F30_GPIO0: J10.3 (Pin_3)
- new net RF4463F30_GPIO1: J11.3 (Pin_3)
- no-connect marks 0 -> 5
Other:
- note removed: "Auf Stm hängen GPIO\n"

Commit message: added powerplane + testpoints + some debugging
Parts:
- added TP8, TP9: TestPoint, STS1library:STS1_Testpoint, symbol Connector:TestPoint
Connections:
- net LoRa_VCC: now also TP8.1
- net RF4463_VCC: now also TP9.1
- net RF4463_nIRQ: no longer names the net of RF2.6 (nIRQ)
- no-connect marks 5 -> 7
Changed lines of the file:
@@
 Connection ~ 2650 3100
 Wire Wire Line
-	2650 3100 2900 3100
+	2650 3100 2750 3100
 Wire Wire Line
 	2900 3200 2900 3100
 Connection ~ 2900 3100
 Wire Wire Line
-	2900 3100 3300 3100
+	2900 3100 3100 3100
 Text HLabel 4400 3800 2    50   Input ~ 0
 LoRa_SPI_CLK
@@
 Connection ~ 7250 3200
 Wire Wire Line
-	7250 3200 7650 3200
+	7250 3200 7550 3200
 $Comp
 L Device:C C15
@@
 Text HLabel 7650 3800 0    50   Input ~ 0
 RF4463_nSEL
-Text HLabel 7650 3700 0    50   Input ~ 0
-RF4463_nIRQ
 Text HLabel 8750 3800 2    50   Input ~ 0
 RF4463_SDI
@@
 Text HLabel 7300 3950 3    50   Input ~ 0
 RF4463F30_SDN
+NoConn ~ 7650 3700
+NoConn ~ 4400 3500
+$Comp
+L Connector:TestPoint TP8
+U 1 1 61B6A550
+P 3100 3100
+F 0 "TP8" H 3050 3400 50  0000 L CNN
+F 1 "TestPoint" H 2950 3300 50  0000 L CNN
+F 2 "STS1library:STS1_Testpoint" H 3300 3100 50  0001 C CNN
+F 3 "~" H 3300 3100 50  0001 C CNN
+	1    3100 3100
+	1    0    0    -1
+$EndComp
+Connection ~ 2750 3100
+Wire Wire Line
+	2750 3100 2900 3100
+$Comp
+L Connector:TestPoint TP9
+U 1 1 61B6AEF9
+P 7550 3200
+F 0 "TP9" H 7500 3500 50  0000 L CNN
+F 1 "TestPoint" H 7400 3400 50  0000 L CNN
+F 2 "STS1library:STS1_Testpoint" H 7750 3200 50  0001 C CNN
+F 3 "~" H 7750 3200 50  0001 C CNN
+	1    7550 3200
+	1    0    0    -1
+$EndComp
+Connection ~ 7550 3200
+Wire Wire Line
+	7550 3200 7650 3200
+Connection ~ 3100 3100
+Wire Wire Line
+	3100 3100 3300 3100
 $EndSCHEMATC

Commit message: finished prototype
Parts:
- R13: value 15 -> 300
Changed lines of the file:
@@
 Connection ~ 2650 3100
-Wire Wire Line
-	2650 3100 2750 3100
 Wire Wire Line
 	2900 3200 2900 3100
@@
 P 3000 4500
 F 0 "R13" H 3070 4546 50  0000 L CNN
-F 1 "15" H 3070 4455 50  0000 L CNN
+F 1 "300" H 3070 4455 50  0000 L CNN
 F 2 "Resistor_SMD:R_0805_2012Metric" V 2930 4500 50  0001 C CNN
 F 3 "~" H 3000 4500 50  0001 C CNN
@@
 	1    0    0    -1
 $EndComp
-Connection ~ 2750 3100
-Wire Wire Line
-	2750 3100 2900 3100
 $Comp
 L Connector:TestPoint TP9
@@
 Wire Wire Line
 	3100 3100 3300 3100
+Wire Wire Line
+	2650 3100 2900 3100
 $EndSCHEMATC
