File: _autosave-STS1_template.kicad_pcb (KiCad board)
At the start: 4 copper layers, 85 x 85 mm, 111 parts, among them IC1 STM32F411RET6TR, IC2 STWD100PYW83F, J10 Conn_01x03_Male, J11 Conn_01x03_Male, J12 Conn_01x03_Male, J2 Conn_01x03_Male, J3 Conn_ARM_JTAG_SWD_10, J39 Conn_Coaxial, J40 Conn_Coaxial, J45 Conn_01x01_Male, J46 Conn_01x01_Male, J5 Conn_01x01_Male, J50 Conn_01x01_Male, J51 Conn_01x01_Male, J52 Conn_01x01_Male, J53 Conn_01x01_Male, J54 Conn_01x01_Male, J55 Conn_01x01_Female, J6 Conn_01x03_Male, J7 Conn_01x03_Male, J8 Conn_01x03_Male, U1 coordinate_system, U2 TPS61288, U3 MCP1725-3302E_MC, Y1 12MHz

Commit message: finished prototype
Parts:
- VCC RF: renamed from TP8
- renumbered TP9 to 5V, TP10 to 5V, TP4 to FRAMCS, TP1 to PA12, TP5 to PB10, TP3 to PB6, TP2 to SWO, TP6 to VCC, TP7 to VCC, TP11 to VCC, TP12 to VCC, TP13 to VCC, TP14 to VCC, TP15 to VCC
Routing:
- net +3V3: track 66.6 -> 79.3 mm

Commit message: COBC v1 (ordered)
Parts:
- moved VCC 1.70 mm to (138.1, 63.6)
Routing:
- net Net-(FLASH1-Pad9): track 5.71 -> 17.3 mm
- net VBUS: track 30.1 -> 38.1 mm
- net +5V: track 150.5 -> 158.4 mm
- net +3V3: track 79.3 -> 87.1 mm, vias 26 -> 19
- net GND: track 78.8 -> 84.8 mm, vias 105 -> 126
- net /EDU_UPDATE: track 102.2 -> 101.0 mm
- net (no net): vias 4 -> 0
- removed copper zone on F.Cu, net +3V3
- removed copper zone on F.Cu, net +5V
- removed copper zone on F.Cu, net Net-(C24-Pad2)
- removed copper zone on F.Cu, net Net-(FLASH1-Pad9)
- removed copper zone on F.Cu, net VBUS
