File: STS1_COBC_uC.kicad_sch (KiCad schematic)
At the start: 42 parts, among them IC2 STWD100PYW83F, IC3 STM32F411RET6TR, J12 Conn_01x01_Male, J13 Conn_01x01_Male, J16 Conn_ARM_JTAG_SWD_10, J17 Conn_01x03_Male, J18 Conn_01x01_Male, J3 Conn_01x01_Male, J4 Conn_01x01_Male, J6 Conn_01x01_Male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

Commit message: ordered version cobc v2
Parts:
- removed J18: Conn_01x01_Male, Connector_PinHeader_2.54mm:PinHeader_1x01_P2.54mm_Vertical, symbol Connector:Conn_01x01_Male
- removed TP18, TP19, TP20: TestPoint, STS1library:STS1_Testpoint, symbol Connector:TestPoint
Connections:
- net PC1 renamed EPS_BAT_FAULT
- net SPI4_NSS: no longer names the net of IC3.33 (PB12)
- no-connect marks 4 -> 5
Changed lines of the file:
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@@
   (junction (at 129.54 50.8) (diameter 0) (color 0 0 0 0)
   )
-  (junction (at 154.94 153.67) (diameter 0) (color 0 0 0 0)
-  )
   (junction (at 62.23 91.44) (diameter 0) (color 0 0 0 0)
   )
@@
   (junction (at 176.53 72.39) (diameter 0) (color 0 0 0 0)
   )
-  (junction (at 152.4 158.75) (diameter 0) (color 0 0 0 0)
-  )
   (junction (at 119.38 105.41) (diameter 0) (color 0 0 0 0)
   )
@@
   (junction (at 116.84 107.95) (diameter 0) (color 0 0 0 0)
   )
-  (junction (at 191.77 115.57) (diameter 0) (color 0 0 0 0)
-  )
   (junction (at 76.2 95.25) (diameter 0) (color 0 0 0 0)
   )
@@
   (junction (at 116.84 121.92) (diameter 0) (color 0 0 0 0)
   )
-  (junction (at 149.86 167.64) (diameter 0) (color 0 0 0 0)
-  )
   (junction (at 125.73 143.51) (diameter 0) (color 0 0 0 0)
   )
@@
   (junction (at 57.15 165.1) (diameter 0) (color 0 0 0 0)
   )
+  (no_connect (at 175.26 115.57))
   (no_connect (at 121.92 110.49))
   (no_connect (at 175.26 107.95))
@@
     (stroke (width 0) (type default) (color 0 0 0 0))
   )
-  (wire (pts (xy 149.86 133.35) (xy 149.86 167.64))
+  (wire (pts (xy 149.86 133.35) (xy 149.86 168.91))
     (stroke (width 0) (type default) (color 0 0 0 0))
   )
@@
     (stroke (width 0) (type default) (color 0 0 0 0))
   )
-  (wire (pts (xy 175.26 115.57) (xy 191.77 115.57))
-    (stroke (width 0) (type default) (color 0 0 0 0))
-  )
   (wire (pts (xy 53.34 25.4) (xy 53.34 22.86))
     (stroke (width 0) (type default) (color 0 0 0 0))
@@
     (stroke (width 0) (type default) (color 0 0 0 0))
   )
-  (wire (pts (xy 154.94 153.67) (xy 154.94 168.91))
+  (wire (pts (xy 154.94 133.35) (xy 154.94 168.91))
     (stroke (width 0) (type default) (color 0 0 0 0))
   )
@@
     (stroke (width 0) (type default) (color 0 0 0 0))
   )
-  (wire (pts (xy 154.94 133.35) (xy 154.94 153.67))
-    (stroke (width 0) (type default) (color 0 0 0 0))
-  )
   (wire (pts (xy 45.72 97.79) (xy 40.64 97.79))
     (stroke (width 0) (type default) (color 0 0 0 0))
@@
     (stroke (width 0) (type default) (color 0 0 0 0))
   )
-  (wire (pts (xy 191.77 115.57) (xy 199.39 115.57))
-    (stroke (width 0) (type default) (color 0 0 0 0))
-  )
   (wire (pts (xy 17.78 167.64) (xy 17.78 165.1))
     (stroke (width 0) (type default) (color 0 0 0 0))
@@
     (stroke (width 0) (type default) (color 0 0 0 0))
   )
-  (wire (pts (xy 121.92 97.79) (xy 119.38 97.79))
+  (wire (pts (xy 113.03 97.79) (xy 121.92 97.79))
     (stroke (width 0) (type default) (color 0 0 0 0))
   )
@@
     (stroke (width 0) (type default) (color 0 0 0 0))
   )
-  (wire (pts (xy 152.4 133.35) (xy 152.4 158.75))
-    (stroke (width 0) (type default) (color 0 0 0 0))
-  )
   (wire (pts (xy 76.2 74.93) (xy 115.57 74.93))
     (stroke (width 0) (type default) (color 0 0 0 0))
@@
     (stroke (width 0) (type default) (color 0 0 0 0))
   )
-  (wire (pts (xy 152.4 158.75) (xy 152.4 168.91))
+  (wire (pts (xy 152.4 133.35) (xy 152.4 168.91))
     (stroke (width 0) (type default) (color 0 0 0 0))
   )
@@
   )
   (wire (pts (xy 17.78 162.56) (xy 24.13 162.56))
-    (stroke (width 0) (type default) (color 0 0 0 0))
-  )
-  (wire (pts (xy 149.86 167.64) (xy 149.86 168.91))
     (stroke (width 0) (type default) (color 0 0 0 0))
   )
@@
     (effects (font (size 1.27 1.27)) (justify right))
   )
-  (hierarchical_label "SPI4_NSS" (shape input) (at 199.39 115.57 0)
-    (effects (font (size 1.27 1.27)) (justify left))
-  )
   (hierarchical_label "EPS_CHARGING" (shape input) (at 40.64 82.55 180)
     (effects (font (size 1.27 1.27)) (justify right))
@@
   )
   (hierarchical_label "EDU_UPDATE" (shape input) (at 154.94 168.91 270)
+    (effects (font (size 1.27 1.27)) (justify right))
+  )
+  (hierarchical_label "EPS_BAT_FAULT" (shape input) (at 113.03 97.79 180)
     (effects (font (size 1.27 1.27)) (justify right))
   )
@@
     (pin "1")
   )
-  (symbol (lib_id "Connector:Conn_01x01_Male") (at 191.77 120.65 90) (unit 1)
-    (in_bom yes) (on_board yes)
-    (property "Reference" "J18" (id 0) (at 194.31 124.46 0))
-    (property "Value" "Conn_01x01_Male" (id 1) (at 191.77 130.81 0))
-    (property "Footprint" "Connector_PinHeader_2.54mm:PinHeader_1x01_P2.54mm_Vertical" (id 2) (at 191.77 120.65 0)
-      (effects (font (size 1.27 1.27)) hide)
-    )
-    (property "Datasheet" "~" (id 3) (at 191.77 120.65 0)
-      (effects (font (size 1.27 1.27)) hide)
-    )
-    (pin "1")
-  )
   (symbol (lib_id "Connector:Conn_ARM_JTAG_SWD_10") (at 72.39 25.4 270) (unit 1)
     (in_bom yes) (on_board yes)
@@
     (pin "2")
   )
-  (symbol (lib_id "Connector:TestPoint") (at 152.4 158.75 270) (unit 1)
-    (in_bom yes) (on_board yes)
-    (property "Reference" "TP19" (id 0) (at 155.3972 160.2232 0)
-      (effects (font (size 1.27 1.27)) (justify left))
-    )
-    (property "Value" "TestPoint" (id 1) (at 153.0858 160.2232 0)
-      (effects (font (size 1.27 1.27)) (justify left))
-    )
-    (property "Footprint" "STS1library:STS1_Testpoint" (id 2) (at 152.4 163.83 0)
-      (effects (font (size 1.27 1.27)) hide)
-    )
-    (property "Datasheet" "~" (id 3) (at 152.4 163.83 0)
-      (effects (font (size 1.27 1.27)) hide)
-    )
-    (pin "1")
-  )
-  (symbol (lib_id "Connector:TestPoint") (at 154.94 153.67 270) (unit 1)
-    (in_bom yes) (on_board yes)
-    (property "Reference" "TP20" (id 0) (at 158.75 148.59 0)
-      (effects (font (size 1.27 1.27)) (justify left))
-    )
-    (property "Value" "TestPoint" (id 1) (at 156.21 144.78 0)
-      (effects (font (size 1.27 1.27)) (justify left))
-    )
-    (property "Footprint" "STS1library:STS1_Testpoint" (id 2) (at 154.94 158.75 0)
-      (effects (font (size 1.27 1.27)) hide)
-    )
-    (property "Datasheet" "~" (id 3) (at 154.94 158.75 0)
-      (effects (font (size 1.27 1.27)) hide)
-    )
-    (pin "1")
-  )
-  (symbol (lib_id "Connector:TestPoint") (at 149.86 167.64 90) (unit 1)
-    (in_bom yes) (on_board yes)
-    (property "Reference" "TP18" (id 0) (at 142.24 170.18 0)
-      (effects (font (size 1.27 1.27)) (justify left))
-    )
-    (property "Value" "TestPoint" (id 1) (at 144.78 172.72 0)
-      (effects (font (size 1.27 1.27)) (justify left))
-    )
-    (property "Footprint" "STS1library:STS1_Testpoint" (id 2) (at 149.86 162.56 0)
-      (effects (font (size 1.27 1.27)) hide)
-    )
-    (property "Datasheet" "~" (id 3) (at 149.86 162.56 0)
-      (effects (font (size 1.27 1.27)) hide)
-    )
-    (pin "1")
-  )
 )

Commit message: Remove old submodules
Connections:
- net SPI_RF_CLK: no longer names the net of IC3.34 (PB13)
- net SPI_RF_MISO: no longer names the net of IC3.44 (PA11)
- net SPI_RF_MOSI: no longer names the net of IC3.15 (PA1)
- no-connect marks 5 -> 8
Changed lines of the file:
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@@
   (no_connect (at 121.92 110.49))
   (no_connect (at 175.26 107.95))
+  (no_connect (at 175.26 113.03))
+  (no_connect (at 175.26 87.63))
   (no_connect (at 175.26 97.79))
+  (no_connect (at 121.92 113.03))
   (no_connect (at 67.31 38.1))
   (wire (pts (xy 17.78 149.86) (xy 24.13 149.86))
@@
     (stroke (width 0) (type default) (color 0 0 0 0))
   )
-  (wire (pts (xy 119.38 113.03) (xy 119.38 129.54))
-    (stroke (width 0) (type default) (color 0 0 0 0))
-  )
   (wire (pts (xy 176.53 44.45) (xy 176.53 72.39))
     (stroke (width 0) (type default) (color 0 0 0 0))
@@
     (stroke (width 0) (type default) (color 0 0 0 0))
   )
-  (wire (pts (xy 121.92 113.03) (xy 119.38 113.03))
-    (stroke (width 0) (type default) (color 0 0 0 0))
-  )
   (wire (pts (xy 53.34 25.4) (xy 53.34 22.86))
     (stroke (width 0) (type default) (color 0 0 0 0))
@@
     (stroke (width 0) (type default) (color 0 0 0 0))
   )
-  (wire (pts (xy 115.57 129.54) (xy 119.38 129.54))
-    (stroke (width 0) (type default) (color 0 0 0 0))
-  )
   (wire (pts (xy 105.41 100.33) (xy 105.41 102.87))
     (stroke (width 0) (type default) (color 0 0 0 0))
@@
     (stroke (width 0) (type default) (color 0 0 0 0))
   )
-  (wire (pts (xy 175.26 87.63) (xy 213.36 87.63))
-    (stroke (width 0) (type default) (color 0 0 0 0))
-  )
   (wire (pts (xy 45.72 149.86) (xy 31.75 149.86))
     (stroke (width 0) (type default) (color 0 0 0 0))
@@
   )
   (wire (pts (xy 129.54 133.35) (xy 80.01 133.35))
-    (stroke (width 0) (type default) (color 0 0 0 0))
-  )
-  (wire (pts (xy 175.26 113.03) (xy 247.65 113.03))
     (stroke (width 0) (type default) (color 0 0 0 0))
   )
@@
     (effects (font (size 1.27 1.27)) (justify left bottom))
   )
-  (label "SPI4_CLK" (at 257.81 74.93 180)
-    (effects (font (size 1.27 1.27)) (justify right bottom))
-  )
-  (label "SPI4_MOSI" (at 115.57 129.54 180)
+  (label "SPI2_CLK" (at 257.81 74.93 180)
     (effects (font (size 1.27 1.27)) (justify right bottom))
   )
@@
     (effects (font (size 1.27 1.27)) (justify left bottom))
   )
-  (label "SPI4_CS_RF" (at 257.81 77.47 180)
-    (effects (font (size 1.27 1.27)) (justify right bottom))
-  )
-  (label "SPI4_MOSI" (at 257.81 72.39 180)
-    (effects (font (size 1.27 1.27)) (justify right bottom))
-  )
-  (label "SPI4_CS_RF" (at 175.26 95.25 0)
+  (label "CS_RF" (at 257.81 77.47 180)
+    (effects (font (size 1.27 1.27)) (justify right bottom))
+  )
+  (label "SPI2_MOSI" (at 257.81 72.39 180)
+    (effects (font (size 1.27 1.27)) (justify right bottom))
+  )
+  (label "SPI2_MOSI" (at 105.41 105.41 180)
+    (effects (font (size 1.27 1.27)) (justify right bottom))
+  )
+  (label "CS_RF" (at 175.26 95.25 0)
     (effects (font (size 1.27 1.27)) (justify left bottom))
   )
@@
     (effects (font (size 1.27 1.27)) (justify right bottom))
   )
-  (label "SPI4_CLK" (at 247.65 113.03 0)
-    (effects (font (size 1.27 1.27)) (justify left bottom))
+  (label "SPI2_MISO" (at 105.41 102.87 180)
+    (effects (font (size 1.27 1.27)) (justify right bottom))
   )
   (label "STM32_NRST" (at 80.01 38.1 0)
@@
     (effects (font (size 1.27 1.27)) (justify right bottom))
   )
-  (label "SPI4_MISO" (at 213.36 87.63 180)
-    (effects (font (size 1.27 1.27)) (justify right bottom))
-  )
   (label "PC1" (at 45.72 97.79 0)
     (effects (font (size 1.27 1.27)) (justify left bottom))
@@
     (effects (font (size 1.27 1.27)) (justify left bottom))
   )
-  (label "SPI4_MISO" (at 257.81 69.85 180)
-    (effects (font (size 1.27 1.27)) (justify right bottom))
-  )
+  (label "SPI2_MISO" (at 257.81 69.85 180)
+    (effects (font (size 1.27 1.27)) (justify right bottom))
+  )
+  (label "SPI2_CLK" (at 99.06 111.76 180)
+    (effects (font (size 1.27 1.27)) (justify right bottom))
+  )

Commit message: V2.5
Parts:
- added D7, D8: LED, LED_SMD:LED_0805_2012Metric, symbol Device:LED
- added JP1: SolderJumper_2_Open, Jumper:SolderJumper-2_P1.3mm_Open_TrianglePad1.0x1.5mm, symbol Jumper:SolderJumper_2_Open
- added R34, R35: 220R, Resistor_SMD:R_0805_2012Metric, symbol Device:R
- J16: footprint STS1library:PinHeader_2x05_P1.27mm_Vertical_SMD -> STS_connector:SAMTEC_FTSH-105-01-X-DH-A
Connections:
- net +3V3: now also JP1.2 (B); no longer J16.1 (VTref)
- net GND: now also D7.1 (K), D8.1 (K)
- net at IC3.33 (PB12): now also R34.1
- net SPI3_CS4: now reaches IC3.34 (PB13)
- net at IC3.36 (PB15): now also R35.1
- new net: J16.1 (VTref), JP1.1 (A)
- new net: D8.2 (A), R35.2
- new net: D7.2 (A), R34.2
- no-connect marks 8 -> 5

Commit message: Set all passive components (except in the RF path) to 0603
Parts:
- C11, C12, C13, C14, C15, C16, C17, C18, C19, C20, C21, C22, C23: footprint Capacitor_SMD:C_0805_2012Metric -> Capacitor_SMD:C_0603_1608Metric
- R1, R3, R34, R35, R4, R5: footprint Resistor_SMD:R_0805_2012Metric -> Resistor_SMD:R_0603_1608Metric
Changed lines of the file:
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@@
       (effects (font (size 1.27 1.27)) (justify left))
     )
-    (property "Footprint" "Capacitor_SMD:C_0805_2012Metric" (id 2) (at 163.5252 140.97 0)
+    (property "Footprint" "Capacitor_SMD:C_0603_1608Metric" (id 2) (at 163.5252 140.97 0)
       (effects (font (size 1.27 1.27)) hide)
     )
@@
     (property "Reference" "C20" (id 0) (at 133.35 41.91 90))
     (property "Value" "100n" (id 1) (at 135.89 45.72 90))
-    (property "Footprint" "Capacitor_SMD:C_0805_2012Metric" (id 2) (at 132.08 44.1452 0)
+    (property "Footprint" "Capacitor_SMD:C_0603_1608Metric" (id 2) (at 132.08 44.1452 0)
       (effects (font (size 1.27 1.27)) hide)
     )
@@
       (effects (font (size 1.27 1.27)) (justify right))
     )
-    (property "Footprint" "Capacitor_SMD:C_0805_2012Metric" (id 2) (at 179.3748 64.77 0)
+    (property "Footprint" "Capacitor_SMD:C_0603_1608Metric" (id 2) (at 179.3748 64.77 0)
       (effects (font (size 1.27 1.27)) hide)
     )
@@
     (property "Reference" "C22" (id 0) (at 172.72 143.51 0))
     (property "Value" "100n" (id 1) (at 172.72 148.59 0))
-    (property "Footprint" "Capacitor_SMD:C_0805_2012Metric" (id 2) (at 173.6852 149.86 0)
+    (property "Footprint" "Capacitor_SMD:C_0603_1608Metric" (id 2) (at 173.6852 149.86 0)
       (effects (font (size 1.27 1.27)) hide)
     )
@@
     (property "Reference" "C18" (id 0) (at 132.08 142.24 90))
     (property "Value" "100n" (id 1) (at 133.35 144.78 90))
-    (property "Footprint" "Capacitor_SMD:C_0805_2012Metric" (id 2) (at 133.35 142.5448 0)
+    (property "Footprint" "Capacitor_SMD:C_0603_1608Metric" (id 2) (at 133.35 142.5448 0)
       (effects (font (size 1.27 1.27)) hide)
     )
@@
       (effects (font (size 1.27 1.27)) (justify left))
     )
-    (property "Footprint" "Resistor_SMD:R_0805_2012Metric" (id 2) (at 80.01 93.472 90)
+    (property "Footprint" "Resistor_SMD:R_0603_1608Metric" (id 2) (at 80.01 93.472 90)
       (effects (font (size 1.27 1.27)) hide)
     )
@@
     (property "Reference" "C17" (id 0) (at 113.03 111.76 0))
     (property "Value" "100n" (id 1) (at 113.03 114.3 0))
-    (property "Footprint" "Capacitor_SMD:C_0805_2012Metric" (id 2) (at 117.8052 115.57 0)
+    (property "Footprint" "Capacitor_SMD:C_0603_1608Metric" (id 2) (at 117.8052 115.57 0)
       (effects (font (size 1.27 1.27)) hide)
     )
@@
     (property "Reference" "C13" (id 0) (at 64.77 86.36 0))
     (property "Value" "20p" (id 1) (at 63.5 86.36 0))
-    (property "Footprint" "Capacitor_SMD:C_0805_2012Metric" (id 2) (at 69.85 85.3948 0)
+    (property "Footprint" "Capacitor_SMD:C_0603_1608Metric" (id 2) (at 69.85 85.3948 0)
       (effects (font (size 1.27 1.27)) hide)
     )
@@
     (property "Reference" "C14" (id 0) (at 64.77 95.25 0))
     (property "Value" "20p" (id 1) (at 63.5 95.25 0))
-    (property "Footprint" "Capacitor_SMD:C_0805_2012Metric" (id 2) (at 69.85 94.2848 0)
+    (property "Footprint" "Capacitor_SMD:C_0603_1608Metric" (id 2) (at 69.85 94.2848 0)
       (effects (font (size 1.27 1.27)) hide)
     )
@@
     (property "Reference" "C19" (id 0) (at 133.35 35.56 90))
     (property "Value" "4.7u" (id 1) (at 135.89 39.37 90))
-    (property "Footprint" "Capacitor_SMD:C_0805_2012Metric" (id 2) (at 132.08 37.7952 0)
+    (property "Footprint" "Capacitor_SMD:C_0603_1608Metric" (id 2) (at 132.08 37.7952 0)
       (effects (font (size 1.27 1.27)) hide)
     )
@@
     (property "Reference" "C16" (id 0) (at 109.22 118.11 0))
     (property "Value" "1u" (id 1) (at 109.22 120.65 0))
-    (property "Footprint" "Capacitor_SMD:C_0805_2012Metric" (id 2) (at 112.0648 114.3 0)
+    (property "Footprint" "Capacitor_SMD:C_0603_1608Metric" (id 2) (at 112.0648 114.3 0)
       (effects (font (size 1.27 1.27)) hide)
     )
@@
       (effects (font (size 1.27 1.27)) (justify right))
     )
-    (property "Footprint" "Resistor_SMD:R_0805_2012Metric" (id 2) (at 27.94 151.638 90)
+    (property "Footprint" "Resistor_SMD:R_0603_1608Metric" (id 2) (at 27.94 151.638 90)
       (effects (font (size 1.27 1.27)) hide)
     )
@@
       (effects (font (size 1.27 1.27)) (justify left))
     )
-    (property "Footprint" "Capacitor_SMD:C_0805_2012Metric" (id 2) (at 53.0352 181.61 0)
+    (property "Footprint" "Capacitor_SMD:C_0603_1608Metric" (id 2) (at 53.0352 181.61 0)
       (effects (font (size 1.27 1.27)) hide)
     )
@@
       (effects (font (size 1.27 1.27)) (justify left))
     )
-    (property "Footprint" "Capacitor_SMD:C_0805_2012Metric" (id 2) (at 58.1152 181.61 0)
+    (property "Footprint" "Capacitor_SMD:C_0603_1608Metric" (id 2) (at 58.1152 181.61 0)
       (effects (font (size 1.27 1.27)) hide)
     )
@@
     (property "Reference" "C15" (id 0) (at 107.95 87.63 0))
     (property "Value" "100n" (id 1) (at 107.95 86.36 0))
-    (property "Footprint" "Capacitor_SMD:C_0805_2012Metric" (id 2) (at 108.9152 92.71 0)
+    (property "Footprint" "Capacitor_SMD:C_0603_1608Metric" (id 2) (at 108.9152 92.71 0)
       (effects (font (size 1.27 1.27)) hide)
     )
@@
       (effects (font (size 1.27 1.27)) (justify left))
     )
-    (property "Footprint" "Resistor_SMD:R_0805_2012Metric" (id 2) (at 206.502 123.825 90)
+    (property "Footprint" "Resistor_SMD:R_0603_1608Metric" (id 2) (at 206.502 123.825 90)
       (effects (font (size 1.27 1.27)) hide)
     )
@@
       (effects (font (size 1.27 1.27)) (justify right))
     )
-    (property "Footprint" "Resistor_SMD:R_0805_2012Metric" (id 2) (at 27.94 144.018 90)
+    (property "Footprint" "Resistor_SMD:R_0603_1608Metric" (id 2) (at 27.94 144.018 90)
       (effects (font (size 1.27 1.27)) hide)
     )
@@
       (effects (font (size 1.27 1.27)) (justify left))
     )
-    (property "Footprint" "Resistor_SMD:R_0805_2012Metric" (id 2) (at 195.072 123.19 90)
+    (property "Footprint" "Resistor_SMD:R_0603_1608Metric" (id 2) (at 195.072 123.19 90)
       (effects (font (size 1.27 1.27)) hide)
     )
@@
       (effects (font (size 1.27 1.27)) (justify right))
     )
-    (property "Footprint" "Resistor_SMD:R_0805_2012Metric" (id 2) (at 208.28 97.028 90)
-      (effects (font (size 1.27 1.27)) hide)
-    )
+    (property "Footprint" "Resistor_SMD:R_0603_1608Metric" (id 2) (at 208.28 97.028 90)
+      (effects (font (size 1.27 1.27)) hide)
+    )

Commit message: Add preliminary resetdog PCB layout.
Connections:
- net DCDC_nEN renamed RDT_CLR
Changed lines of the file:
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@@
     (effects (font (size 1.27 1.27)) (justify right))
   )
-  (hierarchical_label "DCDC_nEN" (shape input) (at 137.16 58.42 90)
+  (hierarchical_label "RDT_CLR" (shape input) (at 137.16 58.42 90)
     (effects (font (size 1.27 1.27)) (justify left))
   )
