File: STS1_COBC_uC.kicad_sch (KiCad schematic)
At the start: 37 parts, among them IC2 STWD100PYW83F, IC3 STM32F411RET6TR, J12 PC0, J13 EPS_Bat_Fault, J16 SWD, J17 Boot0, J3 Conn_01x01_Male, J4 SPI2_CLK, J6 SPI2_MISO, J7 SPI1_CLK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

Commit message: Fix footprint assignments: all IC should have U designator
Parts:
- renumbered IC2 to U18, IC3 to U19
Changed lines of the file:
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@@
   (symbol (lib_id "STS1_COBC_V2-rescue:STM32F411RET6TR-STM32F411RET6TR") (at 121.92 77.47 0) (unit 1)
     (in_bom yes) (on_board yes)
-    (property "Reference" "IC3" (id 0) (at 148.59 92.71 0)
+    (property "Reference" "U19" (id 0) (at 148.59 92.71 0)
       (effects (font (size 1.27 1.27)) (justify left))
     )
@@
   (symbol (lib_id "SamacSys_Parts:STWD100PYW83F") (at 24.13 162.56 0) (unit 1)
     (in_bom yes) (on_board yes)
-    (property "Reference" "IC2" (id 0) (at 38.1 155.829 0))
+    (property "Reference" "U18" (id 0) (at 38.1 155.829 0))
     (property "Value" "STWD100PYW83F" (id 1) (at 38.1 158.1404 0))
     (property "Footprint" "SamacSys_Parts:SOT65P210X110-5N" (id 2) (at 48.26 160.02 0)
