File: uhf_pa.kicad_sch (KiCad schematic)
At the start: 30 parts, among them U12 FPF2701, U13 TQP7M9106

Commit message: feat: clean up schematic
Connections:
- net PA_FAULT renamed PA_Fault
- net RF_IN renamed RF_In
- net RF_OUT renamed RF_Out
- net ~{PA_EN} renamed ~{PA_Enable}
Changed lines of the file:
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@@
     (effects (font (size 1.27 1.27)) (justify right))
   )
-  (hierarchical_label "RF_IN" (shape input) (at 74.93 128.27 180)
+  (hierarchical_label "RF_In" (shape input) (at 74.93 128.27 180)
     (effects (font (size 1.27 1.27)) (justify right))
   )
-  (hierarchical_label "RF_OUT" (shape output) (at 220.98 127 0)
+  (hierarchical_label "RF_Out" (shape output) (at 220.98 127 0)
     (effects (font (size 1.27 1.27)) (justify left))
   )
@@
     (effects (font (size 1.27 1.27)) (justify left))
   )
-  (hierarchical_label "PA_FAULT" (shape output) (at 175.26 52.07 0)
+  (hierarchical_label "PA_Fault" (shape output) (at 175.26 52.07 0)
     (effects (font (size 1.27 1.27)) (justify left))
   )
-  (hierarchical_label "~{PA_EN}" (shape input) (at 113.03 52.07 180)
+  (hierarchical_label "~{PA_Enable}" (shape input) (at 113.03 52.07 180)
     (effects (font (size 1.27 1.27)) (justify right))
   )
-  (symbol (lib_id "power:GND") (at 195.58 138.43 0) (unit 1)
+  (symbol (lib_name "GND_9") (lib_id "power:GND") (at 195.58 138.43 0) (unit 1)
     (in_bom yes) (on_board yes)
     (property "Reference" "#PWR0187" (id 0) (at 195.58 144.78 0)
@@
     (pin "2")
   )
-  (symbol (lib_id "power:GND") (at 151.13 144.78 0) (unit 1)
+  (symbol (lib_name "GND_8") (lib_id "power:GND") (at 151.13 144.78 0) (unit 1)
     (in_bom yes) (on_board yes)
     (property "Reference" "#PWR0186" (id 0) (at 151.13 151.13 0)
@@
     (pin "2")
   )
-  (symbol (lib_id "power:GND") (at 189.23 107.95 0) (unit 1)
+  (symbol (lib_name "GND_1") (lib_id "power:GND") (at 189.23 107.95 0) (unit 1)
     (in_bom yes) (on_board yes)
     (property "Reference" "#PWR0182" (id 0) (at 189.23 114.3 0)
@@
     (pin "1")
   )
-  (symbol (lib_id "power:GND") (at 91.44 138.43 0) (unit 1)
+  (symbol (lib_name "GND_4") (lib_id "power:GND") (at 91.44 138.43 0) (unit 1)
     (in_bom yes) (on_board yes)
     (property "Reference" "#PWR0189" (id 0) (at 91.44 144.78 0)
@@
     (pin "2")
   )
-  (symbol (lib_id "power:GND") (at 165.1 36.83 0) (unit 1)
+  (symbol (lib_name "GND_10") (lib_id "power:GND") (at 165.1 36.83 0) (unit 1)
     (in_bom yes) (on_board yes)
     (property "Reference" "#PWR0191" (id 0) (at 165.1 43.18 0)
@@
     (pin "2")
   )
-  (symbol (lib_id "power:GND") (at 129.54 111.76 0) (unit 1)
+  (symbol (lib_name "GND_2") (lib_id "power:GND") (at 129.54 111.76 0) (unit 1)
     (in_bom yes) (on_board yes)
     (property "Reference" "#PWR0188" (id 0) (at 129.54 118.11 0)
@@
     (pin "1")
   )
-  (symbol (lib_id "power:GND") (at 127 63.5 0) (unit 1)
+  (symbol (lib_name "GND_6") (lib_id "power:GND") (at 127 63.5 0) (unit 1)
     (in_bom yes) (on_board yes)
     (property "Reference" "#PWR0183" (id 0) (at 127 69.85 0)
@@
     (pin "1")
   )
-  (symbol (lib_id "power:GND") (at 151.13 34.29 0) (unit 1)
+  (symbol (lib_name "GND_5") (lib_id "power:GND") (at 151.13 34.29 0) (unit 1)
     (in_bom yes) (on_board yes)
     (property "Reference" "#PWR0185" (id 0) (at 151.13 40.64 0)
@@
     (pin "1")
   )
-  (symbol (lib_id "power:GND") (at 139.7 63.5 0) (unit 1)
+  (symbol (lib_name "GND_7") (lib_id "power:GND") (at 139.7 63.5 0) (unit 1)
     (in_bom yes) (on_board yes)
     (property "Reference" "#PWR0184" (id 0) (at 139.7 69.85 0)
@@
     (pin "9")
   )
-  (symbol (lib_id "power:GND") (at 95.25 110.49 0) (unit 1)
+  (symbol (lib_name "GND_3") (lib_id "power:GND") (at 95.25 110.49 0) (unit 1)
     (in_bom yes) (on_board yes)
     (property "Reference" "#PWR0190" (id 0) (at 95.25 116.84 0)
