File: uhf_pa.kicad_sch (KiCad schematic)
At the start: 26 parts, among them U12 TPS22950_Q1, U13 TQP7M9106

Commit message: fix: use 0805 size inductor for PA power supply and make DRC happy after KiCAD10 upgrade
Parts:
- L17: footprint Inductor_SMD:L_0402_1005Metric -> Inductor_SMD:L_0805_2012Metric; JLCPCB Part # C344018 -> C2042168; Manufacturer_Part_Number LQW15AN18NJ80D -> LQW2BAN18NG00L; PartNumber LQW15AN18NJ80D -> LQW2BAN18NG00L
- TP7: footprint TestPoint:TestPoint_Keystone_5015_Micro-Minature -> TestPoint:TestPoint_Keystone_5015_Micro_Mini
Changed lines of the file:
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@@
 			)
 		)
-		(property "Footprint" "Inductor_SMD:L_0402_1005Metric"
+		(property "Footprint" "Inductor_SMD:L_0805_2012Metric"
 			(at 175.26 123.19 0)
 			(hide yes)
@@
 			)
 		)
-		(property "PartNumber" "LQW15AN18NJ80D"
+		(property "PartNumber" "LQW2BAN18NG00L"
 			(at 175.26 123.19 0)
 			(hide yes)
@@
 			)
 		)
-		(property "JLCPCB Part #" "C344018"
+		(property "JLCPCB Part #" "C2042168"
 			(at 175.26 123.19 0)
 			(hide yes)
@@
 			)
 		)
-		(property "Manufacturer_Part_Number" "LQW15AN18NJ80D "
+		(property "Manufacturer_Part_Number" "LQW2BAN18NG00L"
 			(at 175.26 123.19 0)
 			(hide yes)
@@
 			)
 		)
-		(property "Footprint" "TestPoint:TestPoint_Keystone_5015_Micro-Minature"
+		(property "Footprint" "TestPoint:TestPoint_Keystone_5015_Micro_Mini"
 			(at 158.75 147.32 0)
 			(hide yes)
