File: LatchUp.kicad_sch (KiCad schematic)
At the start: 25 parts, among them Q10 IRF7406, Q11 BSL307SP, Q9 BSS138, U25 INA138NA_3K, U26 AD589JRZ, U27 LT1636CMS8_PBF

Commit message: Add manufacture number and JLCPCB part number to components
Parts:
- C90, C92: JLCPCB Part # (none) -> C1591; Manufacturer_Part_Number (none) -> CL10B104KB8NNNC
- C91: JLCPCB Part # (none) -> C3876314; Manufacturer_Part_Number (none) -> CL10C220JB8NNWC
- D17, D20: JLCPCB Part # (none) -> C83528; Manufacturer_Part_Number (none) -> 1N4148W-7-F
- D18: Manufacturer_Part_Number (none) -> BZY55C2V7 RBG
- D19: JLCPCB Part # (none) -> C131660; Manufacturer_Part_Number (none) -> BZX84-C16,215
- D21, D22: JLCPCB Part # (none) -> C550933; Manufacturer_Part_Number (none) -> BZX84-C10,235
- Q10: JLCPCB Part # (none) -> C169769; Manufacturer_Part_Number (none) -> IRF7406TRPBF
- Q11: JLCPCB Part # (none) -> C534457; Manufacturer_Part_Number (none) -> BSL307SP H6327
- Q9: JLCPCB Part # (none) -> C52895; Manufacturer_Part_Number (none) -> BSS138
- R59: JLCPCB Part # (none) -> C327839; Manufacturer_Part_Number (none) -> MR06X4703FTL
- R60: JLCPCB Part # (none) -> C4247597; Manufacturer_Part_Number (none) -> ERJ-H3EF2702V
- R61: JLCPCB Part # (none) -> C4117710; Manufacturer_Part_Number (none) -> ERJ-H3G0R00V
- R62, R63: Manufacturer_Part_Number (none) -> MR06X1004FTL
- R64, R65, R67: JLCPCB Part # (none) -> C4220470; Manufacturer_Part_Number (none) -> ERJ-H3EF3302V
- R66: Manufacturer_Part_Number (none) -> MR06X3303FTL
- U25: JLCPCB Part # (none) -> C47914; Manufacturer_Part_Number (none) -> INA138NA/3K
- U26: JLCPCB Part # (none) -> C207416; Manufacturer_Part_Number (none) -> AD589JRZ-REEL
- U27: JLCPCB Part # (none) -> C579794; MANUFACTURER_PART_NUMBER LT1636CMS8#PBF -> (none); Manufacturer_Part_Number (none) -> LT1636CMS8#PBF
