File: LatchUp.kicad_sch (KiCad schematic)
At the start: 27 parts, among them Q5 BSS138, Q6 IRF7406, Q7 BSL307SP, U21 INA138NA_3K, U22 AD589JRZ, U23 LT1636CMS8_PBF

Commit message: Mark do-no-populate components as such
Parts:
- D13, R50: now not fitted
Other:
- note removed: "DNP"
Changed lines of the file:
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@@
 	(generator_version "10.0")
 	(paper "A4")
-	(text "DNP"
-		(exclude_from_sim no)
-		(at 235.458 100.33 0)
-		(effects
-			(font
-				(size 1.27 1.27)
-			)
-			(justify left bottom)
-		)
-	)
-	(text "DNP"
-		(exclude_from_sim no)
-		(at 217.17 98.044 0)
-		(effects
-			(font
-				(size 1.27 1.27)
-			)
-			(justify left bottom)
-		)
-	)
 	(text "The following schematics is comming from the thesis\n\"Project solutions for low-cost space missions\" by Stefano Speretta\nhttps://zerorobotics.polito.it/app/uploads/2019/04/thesis-1.pdf"
 		(exclude_from_sim no)
@@
 		)
 	)
-	(polyline
-		(pts
-			(xy 229.87 97.79) (xy 240.03 97.79)
-		)
-		(stroke
-			(width 0)
-			(type dash)
-		)
-	)
 	(wire
 		(pts
@@
 		)
 	)
-	(polyline
-		(pts
-			(xy 229.87 106.68) (xy 240.03 106.68)
-		)
-		(stroke
-			(width 0)
-			(type dash)
-		)
-	)
 	(wire
 		(pts
@@
 		)
 	)
-	(polyline
-		(pts
-			(xy 212.09 95.25) (xy 212.09 104.14)
-		)
-		(stroke
-			(width 0)
-			(type dash)
-		)
-	)
 	(wire
 		(pts
@@
 		)
 	)
-	(polyline
-		(pts
-			(xy 212.09 95.25) (xy 224.79 95.25)
-		)
-		(stroke
-			(width 0)
-			(type dash)
-		)
-	)
 	(wire
 		(pts
@@
 		)
 	)
-	(polyline
-		(pts
-			(xy 229.87 97.79) (xy 229.87 106.68)
-		)
-		(stroke
-			(width 0)
-			(type dash)
-		)
-	)
 	(wire
 		(pts
@@
 		)
 	)
-	(polyline
-		(pts
-			(xy 224.79 104.14) (xy 224.79 95.25)
-		)
-		(stroke
-			(width 0)
-			(type dash)
-		)
-	)
 	(wire
 		(pts
@@
 		)
 	)
-	(polyline
-		(pts
-			(xy 212.09 104.14) (xy 224.79 104.14)
-		)
-		(stroke
-			(width 0)
-			(type dash)
-		)
-	)
-	(polyline
-		(pts
-			(xy 240.03 106.68) (xy 240.03 97.79)
-		)
-		(stroke
-			(width 0)
-			(type dash)
-		)
-	)
 	(wire
 		(pts
@@
 		(on_board no)
 		(in_pos_files yes)
-		(dnp no)
+		(dnp yes)
 		(fields_autoplaced yes)
 		(property "Reference" "R50"
@@
 		(on_board no)
 		(in_pos_files yes)
-		(dnp no)
+		(dnp yes)
 		(fields_autoplaced yes)
 		(property "Reference" "D13"
