File: Resetdog.kicad_sch (KiCad schematic)
At the start: 20 parts, among them U14 MC14541BD, U15 MC74HC4538ADG, U20 74LVC1G17

Commit message: Mark do-no-populate components as such
Parts:
- R111: now not fitted
Other:
- note removed: "DNP"
Changed lines of the file:
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@@
-		)
-	)
-	(text "DNP"
-		(exclude_from_sim no)
-		(at 31.75 82.55 0)
-		(effects
-			(font
-				(size 1.27 1.27)
-			)
-			(justify left bottom)
 		)
 	)
@@
 		)
 	)
-	(polyline
-		(pts
-			(xy 29.21 80.01) (xy 29.21 86.36)
-		)
-		(stroke
-			(width 0)
-			(type dash)
-		)
-	)
 	(wire
 		(pts
@@
 		)
 	)
-	(polyline
-		(pts
-			(xy 29.21 86.36) (xy 40.64 86.36)
-		)
-		(stroke
-			(width 0)
-			(type dash)
-		)
-	)
 	(wire
 		(pts
@@
 		)
 	)
-	(polyline
-		(pts
-			(xy 29.21 80.01) (xy 40.64 80.01)
-		)
-		(stroke
-			(width 0)
-			(type dash)
-		)
-	)
 	(wire
 		(pts
@@
 			(width 0)
 			(type default)
-		)
-	)
-	(polyline
-		(pts
-			(xy 40.64 86.36) (xy 40.64 80.01)
-		)
-		(stroke
-			(width 0)
-			(type dash)
 		)
 	)
@@
 		(on_board yes)
 		(in_pos_files yes)
-		(dnp no)
+		(dnp yes)
 		(property "Reference" "R111"
 			(at 35.56 82.55 90)
