File: STS1_COBC.kicad_pcb (KiCad board)
At the start: 4 copper layers, 81 x 85 mm, 328 parts, among them J1 UHF, J16 SWD, Q1 SQ2318, Q10 IRF7406, Q11 BSL307SP, Q12 BSS123, Q13 BSS123, Q2 BSS123, Q3 SQ2318, Q4 SQ2318, Q5 BSS138, Q6 IRF7406, Q7 BSL307SP, Q8 BSS123, Q9 BSS138, U1 W25Q01JVZEIQ, U10 TQP3M9036, U11 74LVC1G14Z-7, U12 TPS22950_Q1, U13 TQP7M9106, U14 MC14541BD, U15 MC74HC4538ADG, U16 F2972, U17 CY15B104Q-SXI, U18 STWD100PYW83F, U19 STM32F411RET6TR, U2 LP2985-1.8, U20 74LVC1G17, U21 INA138NA_3K, U22 AD589JRZ, U23 LT1636CMS8_PBF, U24 MCP1725-3302E_MC, U25 INA138NA_3K, U26 AD589JRZ, U27 LT1636CMS8_PBF, U28 MCP130T-300I_TT, U29 74LVC1G08GV,125, U3 MCP1725-3302E_MC, U30 TMP36xS, U31 74LVC1G08GV,125, U32 74LVC1G32GV,125, U4 74LVC2G74, U5 TYKTBCSANF-26.000000, U6 MP28167GQ, U8 Si4463, U9 LFCG-490+, Y1 12M

Commit message: fix: update coordinate system
Parts:
- turned CS1 to 0 degrees
